Commit message: Added DEV kits | applied tests
Signed-off-by: Jakub Delicat <jakub.delicat@husarion.com>

File: urdf/components.urdf.xacro (robot description, xacro)
@@ -17,242 +17,267 @@
       <xacro:property name="index" value="${counter - 1}" scope="parent" />
       <xacro:property name="component" value="${config['components'][index]}" scope="parent" />
-      <xacro:property name="type" value="${component['type']}" scope="parent" />
-      <xacro:property name="parent_link" value="${component['parent_link']}" scope="parent" />
-      <xacro:property name="xyz" value="${component['xyz']}" scope="parent" />
-      <xacro:property name="rpy" value="${component['rpy']}" scope="parent" />
-      <xacro:if value="${robot_namespace == ''}">
-        <xacro:property name="ns" value="None" scope="parent" />
-      </xacro:if>
-      <xacro:unless value="${robot_namespace == ''}">
-        <xacro:property name="ns" value="${robot_namespace}" scope="parent" />
-      </xacro:unless>
-      <xacro:if value="${'device_namespace' in component}">
-        <xacro:property name="device_namespace" value="${component['device_namespace']}" scope="parent" />
-      </xacro:if>
-      <xacro:unless value="${'device_namespace' in component}">
-        <xacro:property name="device_namespace" value="" scope="parent" />
-      </xacro:unless>
-      <xacro:if value="${type == 'ANT02'}">
+        <xacro:if value="${robot_namespace == ''}">
+          <xacro:property name="ns" value="None" scope="parent" />
+        </xacro:if>
+        <xacro:unless value="${robot_namespace == ''}">
+          <xacro:property name="ns" value="${robot_namespace}" scope="parent" />
+        </xacro:unless>
+        <xacro:property name="type" value="${component['type']}" scope="parent" />
+        <xacro:property name="dev_models_dict"
+          value="${dict ([
+          ('DEV01', 'dev01'),
+          ('DEV02', 'dev02'),
+          ('DEV03', 'dev03'),
+          ('DEV04H', 'dev04h'),
+          ('DEV04L', 'dev04l'),
+          ('DEV05', 'dev05'),
+          ('DEV06', 'dev06'),
+          ('DEV07', 'dev07'),
+          ('DEV07T', 'dev07t'),
+          ('DEV09', 'dev09')
+        ])}" />
+      <xacro:if value="${type in dev_models_dict}">
         <xacro:include
-          filename="$(find ros_components_description)/urdf/teltonika_003R-00253.urdf.xacro"
-          ns="teltonika" />
-        <xacro:teltonika.teltonika_003R-00253
-          parent_link="${parent_link}"
-          xyz="${xyz}"
-          rpy="${rpy}"
+          filename="$(find ros_components_description)/urdf/dev.urdf.xacro"
+          ns="dev"
+        />
+        <xacro:dev.dev
           namespace="${ns}"
-          device_namespace="${device_namespace}"
+          model="${dev_models_dict[type]}"
         />
       </xacro:if>
-      <xacro:if value="${type == 'CAM01'}">
-        <xacro:include
-          filename="$(find ros_components_description)/urdf/orbbec_astra.urdf.xacro"
-          ns="camera" />
-        <xacro:if value="${device_namespace == ''}">
-          <xacro:property name="device_namespace" value="camera" scope="parent" />
-        </xacro:if>
-        <xacro:camera.orbbec_astra
-          parent_link="${parent_link}"
-          xyz="${xyz}"
-          rpy="${rpy}"
-          namespace="${ns}"
-          device_namespace="${device_namespace}"
-        />
-      </xacro:if>
-      <xacro:property name="zed_models_dict"
-        value="${dict ([
-        ('CAM03', 'zed2'),
-        ('CAM04', 'zed2i'),
-        ('CAM06', 'zedx'),
+      <xacro:unless value="${type in dev_models_dict}">
+        <xacro:property name="parent_link" value="${component['parent_link']}" scope="parent" />
+        <xacro:property name="xyz" value="${component['xyz']}" scope="parent" />
+        <xacro:property name="rpy" value="${component['rpy']}" scope="parent" />
+        <xacro:if value="${'device_namespace' in component}">
+          <xacro:property name="device_namespace" value="${component['device_namespace']}" scope="parent" />
+        </xacro:if>
+        <xacro:unless value="${'device_namespace' in component}">
+          <xacro:property name="device_namespace" value="" scope="parent" />
+        </xacro:unless>
+        <xacro:if value="${type == 'ANT02'}">
+          <xacro:include
+            filename="$(find ros_components_description)/urdf/teltonika_003R-00253.urdf.xacro"
+            ns="teltonika" />
+          <xacro:teltonika.teltonika_003R-00253
+            parent_link="${parent_link}"
+            xyz="${xyz}"
+            rpy="${rpy}"
+            namespace="${ns}"
+            device_namespace="${device_namespace}"
+          />
+        </xacro:if>
+        <xacro:if value="${type == 'CAM01'}">
+          <xacro:include
+            filename="$(find ros_components_description)/urdf/orbbec_astra.urdf.xacro"
+            ns="camera" />
+          <xacro:if value="${device_namespace == ''}">
+            <xacro:property name="device_namespace" value="camera" scope="parent" />
+          </xacro:if>
+          <xacro:camera.orbbec_astra
+            parent_link="${parent_link}"
+            xyz="${xyz}"
+            rpy="${rpy}"
+            namespace="${ns}"
+            device_namespace="${device_namespace}"
+          />
+        </xacro:if>
+        <xacro:property name="zed_models_dict"
+          value="${dict ([
+          ('CAM03', 'zed2'),
+          ('CAM04', 'zed2i'),
+          ('CAM06', 'zedx'),
+          ])}" />
+          <xacro:if value="${type in zed_models_dict}">
+          <xacro:include
+            filename="$(find ros_components_description)/urdf/stereolabs_zed.urdf.xacro"
+            ns="camera" />
+          <xacro:if value="${device_namespace == ''}">
+            <xacro:property name="device_namespace" value="zed" scope="parent" />
+          </xacro:if>
+          <xacro:camera.zed_camera
+            parent_link="${parent_link}"
+            xyz="${xyz}"
+            rpy="${rpy}"
+            namespace="${ns}"
+            device_namespace="${device_namespace}"
+            model="${zed_models_dict[type]}"
+          />
+        </xacro:if>
+        <xacro:property name="rplidar_models_dict"
+          value="${dict ([
+          ('LDR01', 's1'),
+          ('LDR06', 's3'),
         ])}" />
-        <xacro:if value="${type in zed_models_dict}">
-        <xacro:include
-          filename="$(find ros_components_description)/urdf/stereolabs_zed.urdf.xacro"
-          ns="camera" />
-        <xacro:if value="${device_namespace == ''}">
-          <xacro:property name="device_namespace" value="zed" scope="parent" />
-        </xacro:if>
-        <xacro:camera.zed_camera
-          parent_link="${parent_link}"
-          xyz="${xyz}"
-          rpy="${rpy}"
-          namespace="${ns}"
-          device_namespace="${device_namespace}"
-          model="${zed_models_dict[type]}"
-        />
-      </xacro:if>
-      <xacro:property name="rplidar_models_dict"
-        value="${dict ([
-        ('LDR01', 's1'),
-        ('LDR06', 's3'),
-      ])}" />
-      <xacro:if value="${type in rplidar_models_dict}">
-        <xacro:include
-          filename="$(find ros_components_description)/urdf/slamtec_rplidar.urdf.xacro"
-          ns="lidar"
-        />
-        <xacro:lidar.slamtec_rplidar
-          parent_link="${parent_link}"
-          xyz="${xyz}"
-          rpy="${rpy}"
-          namespace="${ns}"
-          device_namespace="${device_namespace}"
-          model="${rplidar_models_dict[type]}"
-        />
-      </xacro:if>
-      <xacro:property name="ouster_models_dict"
-        value="${dict ([
-        ('LDR10', 'os0_32'),
-        ('LDR11', 'os0_64'),
-        ('LDR12', 'os0_128'),
-        ('LDR13', 'os1_32'),
-        ('LDR14', 'os1_64'),
-        ('LDR15', 'os1_128')
-      ])}" />
-      <xacro:if value="${type in ouster_models_dict}">
-        <xacro:include
-          filename="$(find ros_components_description)/urdf/ouster.urdf.xacro"
-          ns="lidar"
-        />
-        <xacro:lidar.ouster
-          parent_link="${parent_link}"
-          xyz="${xyz}"
-          rpy="${rpy}"
-          namespace="${ns}"
-          device_namespace="${device_namespace}"
-          model="${ouster_models_dict[type]}"
-        />
-      </xacro:if>
-      <xacro:if value="${type == 'LDR20'}">
-        <xacro:include
-          filename="$(find ros_components_description)/urdf/velodyne_puck.urdf.xacro"
-          ns="lidar"
-        />
-        <xacro:lidar.velodyne_puck
-          parent_link="${parent_link}"
-          xyz="${xyz}"
-          rpy="${rpy}"
-          namespace="${ns}"
-          device_namespace="${device_namespace}"
-        />
-      </xacro:if>
-      <xacro:if value="${type == 'MAN01'}">
-        <xacro:include
-          filename="$(find ros_components_description)/urdf/ur.urdf.xacro"
-          ns="manipulator"
-        />
-        <xacro:manipulator.ur
-          parent_link="${parent_link}"
-          xyz="${xyz}"
-          rpy="${rpy}"
-          device_namespace="${device_namespace}"
-          ur_type="ur3e"
-        />
-      </xacro:if>
-      <xacro:if value="${type == 'MAN02'}">
-        <xacro:include
-          filename="$(find ros_components_description)/urdf/ur.urdf.xacro"
-          ns="manipulator"
-        />
-        <xacro:manipulator.ur
-          parent_link="${parent_link}"
-          xyz="${xyz}"
-          rpy="${rpy}"
-          device_namespace="${device_namespace}"
-          ur_type="ur5e"
-        />
-      </xacro:if>
-      <xacro:if value="${type == 'MAN04'}">
-        <xacro:include
-          filename="$(find ros_components_description)/urdf/kinova.urdf.xacro"
-          ns="manipulator"
-        />
-        <xacro:manipulator.kinova
-          parent_link="${parent_link}"
-          xyz="${xyz}"
-          rpy="${rpy}"
-          namespace="${ns}"
-          device_namespace="${device_namespace}"
-          kinova_type="gen3"
-          dof="6"
-          gripper="robotiq_2f_85"
-          vision="false"
-        />
-      </xacro:if>
-      <xacro:if value="${type == 'MAN05'}">
-        <xacro:include
-          filename="$(find ros_components_description)/urdf/kinova.urdf.xacro"
-          ns="manipulator"
-        />
-        <xacro:manipulator.kinova
-          parent_link="${parent_link}"
-          xyz="${xyz}"
-          rpy="${rpy}"
-          namespace="${ns}"
-          device_namespace="${device_namespace}"
-          kinova_type="gen3"
-          dof="6"
-          gripper="robotiq_2f_85"
-          vision="true"
-        />
-      </xacro:if>
-      <xacro:if value="${type == 'MAN06'}">
-        <xacro:include
-          filename="$(find ros_components_description)/urdf/kinova.urdf.xacro"
-          ns="manipulator"
-        />
-        <xacro:manipulator.kinova
-          parent_link="${parent_link}"
-          xyz="${xyz}"
-          rpy="${rpy}"
-          namespace="${ns}"
-          device_namespace="${device_namespace}"
-          kinova_type="gen3"
-          dof="7"
-          gripper="robotiq_2f_85"
-          vision="false"
-        />
-      </xacro:if>
-      <xacro:if value="${type == 'MAN07'}">
-        <xacro:include
-          filename="$(find ros_components_description)/urdf/kinova.urdf.xacro"
-          ns="manipulator"
-        />
-        <xacro:manipulator.kinova
-          parent_link="${parent_link}"
-          xyz="${xyz}"
-          rpy="${rpy}"
-          namespace="${ns}"
-          kinova_type="gen3"
-          dof="7"
-          gripper="robotiq_2f_85"
-          vision="true"
-          device_namespace="${device_namespace}"
-        />
-      </xacro:if>
-      <xacro:if value="${type == 'GRP02'}">
-        <xacro:include filename="$(find ros_components_description)/urdf/robotiq.urdf.xacro"
-          ns="gripper" />
-        <xacro:gripper.robotiq
-          parent_link="${parent_link}"
-          xyz="${xyz}"
-          rpy="${rpy}"
-          namespace="${ns}"
-          device_namespace="${device_namespace}"
-          robotiq_type="2f_85"
-        />
-      </xacro:if>
-      <xacro:if value="${type == 'WCH01'}">
-        <xacro:include
-          filename="$(find ros_components_description)/urdf/wibotic_receiver.urdf.xacro"
-          ns="wireless_charger" />
-        <xacro:wireless_charger.wibotic_receiver
-          parent_link="${parent_link}"
-          xyz="${xyz}"
-          rpy="${rpy}"
-          namespace="${ns}"
-          device_namespace="${device_namespace}"
-        />
-      </xacro:if>
+        <xacro:if value="${type in rplidar_models_dict}">
+          <xacro:include
+            filename="$(find ros_components_description)/urdf/slamtec_rplidar.urdf.xacro"
+            ns="lidar"
+          />
+          <xacro:lidar.slamtec_rplidar
+            parent_link="${parent_link}"
+            xyz="${xyz}"
+            rpy="${rpy}"
+            namespace="${ns}"
+            device_namespace="${device_namespace}"
+            model="${rplidar_models_dict[type]}"
+          />
+        </xacro:if>
+        <xacro:property name="ouster_models_dict"
+          value="${dict ([
+          ('LDR10', 'os0_32'),
+          ('LDR11', 'os0_64'),
+          ('LDR12', 'os0_128'),
+          ('LDR13', 'os1_32'),
+          ('LDR14', 'os1_64'),
+          ('LDR15', 'os1_128')
+        ])}" />
+        <xacro:if value="${type in ouster_models_dict}">
+          <xacro:include
+            filename="$(find ros_components_description)/urdf/ouster.urdf.xacro"
+            ns="lidar"
+          />
+          <xacro:lidar.ouster
+            parent_link="${parent_link}"
+            xyz="${xyz}"
+            rpy="${rpy}"
+            namespace="${ns}"
+            device_namespace="${device_namespace}"
+            model="${ouster_models_dict[type]}"
+          />
+        </xacro:if>
+        <xacro:if value="${type == 'LDR20'}">
+          <xacro:include
+            filename="$(find ros_components_description)/urdf/velodyne_puck.urdf.xacro"
+            ns="lidar"
+          />
+          <xacro:lidar.velodyne_puck
+            parent_link="${parent_link}"
+            xyz="${xyz}"
+            rpy="${rpy}"
+            namespace="${ns}"
+            device_namespace="${device_namespace}"
+          />
+        </xacro:if>
+        <xacro:if value="${type == 'MAN01'}">
+          <xacro:include
+            filename="$(find ros_components_description)/urdf/ur.urdf.xacro"
+            ns="manipulator"
+          />
+          <xacro:manipulator.ur
+            parent_link="${parent_link}"
+            xyz="${xyz}"
+            rpy="${rpy}"
+            device_namespace="${device_namespace}"
+            ur_type="ur3e"
+          />
+        </xacro:if>
+        <xacro:if value="${type == 'MAN02'}">
+          <xacro:include
+            filename="$(find ros_components_description)/urdf/ur.urdf.xacro"
+            ns="manipulator"
+          />
+          <xacro:manipulator.ur
+            parent_link="${parent_link}"
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