Commit message: Added all DEVs to tests | fixed DEV09
Signed-off-by: Jakub Delicat <jakub.delicat@husarion.com>

File: urdf/dev.urdf.xacro (robot description, xacro)
@@ -83,4 +83,12 @@
       <xacro:property name="collision_box_xyz"  value="0 0 0.07"      scope="parent" />
     </xacro:if>
+    <xacro:if value="${model == 'dev09'}">
+      <xacro:property name="parent_link" value="mount_link" scope="parent" />
+      <xacro:property name="xyz" value="0 0 0"  scope="parent" />
+      <xacro:property name="rpy" value="0 0 ${-pi/2.0}" scope="parent" />
+      <xacro:property name="collision_box_size" value="0.235 0.525 0.25"      scope="parent" />
+      <xacro:property name="collision_box_rpy"  value="0 0 ${-pi/2.0}"      scope="parent" />
+      <xacro:property name="collision_box_xyz"  value="0 0 0.125"      scope="parent" />
+    </xacro:if>
     <joint name="${ns}${model}_joint" type="fixed">
       <origin xyz="${xyz}" rpy="${rpy}" />
