Commit message: minor fix

File: test/component.urdf.xacro (robot description, xacro)
@@ -5,5 +5,5 @@
   <xacro:property name="components_config_path_property" value="$(arg components_config_path)" />
   <xacro:if value="${components_config_path_property != ''}">
-    <xacro:include filename="$(find ros_components_description)/urdf/components.urdf.xacro" ns="husarion_components" />
+    <xacro:include filename="$(find psd_sensors)/urdf/components.urdf.xacro" ns="husarion_components" />
     <xacro:husarion_components.create_components
       components_config_path="${components_config_path_property}"

File: urdf/components.urdf.xacro (robot description, xacro)
@@ -24,5 +24,5 @@
       <xacro:if value="${type == 'ANT02'}">
         <xacro:include
-          filename="$(find ros_components_description)/urdf/teltonika_003R-00253.urdf.xacro"
+          filename="$(find psd_sensors)/urdf/teltonika_003R-00253.urdf.xacro"
           ns="teltonika" />
         <xacro:teltonika.teltonika_003R-00253
@@ -36,5 +36,5 @@
       <xacro:if value="${type == 'CAM01'}">
         <xacro:include
-          filename="$(find ros_components_description)/urdf/orbbec_astra.urdf.xacro"
+          filename="$(find psd_sensors)/urdf/orbbec_astra.urdf.xacro"
           ns="camera" />
         <xacro:if value="${device_ns == ''}">
@@ -57,5 +57,5 @@
         <xacro:if value="${type in zed_models_dict}">
         <xacro:include
-          filename="$(find ros_components_description)/urdf/stereolabs_zed.urdf.xacro"
+          filename="$(find psd_sensors)/urdf/stereolabs_zed.urdf.xacro"
           ns="camera" />
         <xacro:if value="${device_ns == ''}">
@@ -73,5 +73,5 @@
       <xacro:if value="${type == 'CAM11'}">
         <xacro:include
-          filename="$(find ros_components_description)/urdf/luxonis_depthai.urdf.xacro"
+          filename="$(find psd_sensors)/urdf/luxonis_depthai.urdf.xacro"
           ns="camera" />
         <xacro:if value="${device_ns == ''}">
@@ -95,5 +95,5 @@
       <xacro:if value="${type in rplidar_models_dict}">
         <xacro:include
-          filename="$(find ros_components_description)/urdf/slamtec_rplidar.urdf.xacro"
+          filename="$(find psd_sensors)/urdf/slamtec_rplidar.urdf.xacro"
           ns="lidar"
         />
@@ -118,5 +118,5 @@
       <xacro:if value="${type in ouster_models_dict}">
         <xacro:include
-          filename="$(find ros_components_description)/urdf/ouster.urdf.xacro"
+          filename="$(find psd_sensors)/urdf/ouster.urdf.xacro"
           ns="lidar"
         />
@@ -132,5 +132,5 @@
       <xacro:if value="${type == 'LDR20'}">
         <xacro:include
-          filename="$(find ros_components_description)/urdf/velodyne_puck.urdf.xacro"
+          filename="$(find psd_sensors)/urdf/velodyne_puck.urdf.xacro"
           ns="lidar"
         />
@@ -145,5 +145,5 @@
       <xacro:if value="${type == 'MAN01'}">
         <xacro:include
-          filename="$(find ros_components_description)/urdf/ur.urdf.xacro"
+          filename="$(find psd_sensors)/urdf/ur.urdf.xacro"
           ns="manipulator"
         />
@@ -158,5 +158,5 @@
       <xacro:if value="${type == 'MAN02'}">
         <xacro:include
-          filename="$(find ros_components_description)/urdf/ur.urdf.xacro"
+          filename="$(find psd_sensors)/urdf/ur.urdf.xacro"
           ns="manipulator"
         />
@@ -171,5 +171,5 @@
       <xacro:if value="${type == 'MAN04'}">
         <xacro:include
-          filename="$(find ros_components_description)/urdf/kinova.urdf.xacro"
+          filename="$(find psd_sensors)/urdf/kinova.urdf.xacro"
           ns="manipulator"
         />
@@ -188,5 +188,5 @@
       <xacro:if value="${type == 'MAN05'}">
         <xacro:include
-          filename="$(find ros_components_description)/urdf/kinova.urdf.xacro"
+          filename="$(find psd_sensors)/urdf/kinova.urdf.xacro"
           ns="manipulator"
         />
@@ -205,5 +205,5 @@
       <xacro:if value="${type == 'MAN06'}">
         <xacro:include
-          filename="$(find ros_components_description)/urdf/kinova.urdf.xacro"
+          filename="$(find psd_sensors)/urdf/kinova.urdf.xacro"
           ns="manipulator"
         />
@@ -222,5 +222,5 @@
       <xacro:if value="${type == 'MAN07'}">
         <xacro:include
-          filename="$(find ros_components_description)/urdf/kinova.urdf.xacro"
+          filename="$(find psd_sensors)/urdf/kinova.urdf.xacro"
           ns="manipulator"
         />
@@ -238,5 +238,5 @@
       </xacro:if>
       <xacro:if value="${type == 'GRP02'}">
-        <xacro:include filename="$(find ros_components_description)/urdf/robotiq.urdf.xacro"
+        <xacro:include filename="$(find psd_sensors)/urdf/robotiq.urdf.xacro"
           ns="gripper" />
         <xacro:gripper.robotiq
@@ -251,5 +251,5 @@
       <xacro:if value="${type == 'WCH01'}">
         <xacro:include
-          filename="$(find ros_components_description)/urdf/wibotic_receiver.urdf.xacro"
+          filename="$(find psd_sensors)/urdf/wibotic_receiver.urdf.xacro"
           ns="wireless_charger" />
         <xacro:wireless_charger.wibotic_receiver

File: urdf/intel_realsense_d435.urdf.xacro (robot description, xacro)
@@ -67,5 +67,5 @@
         <origin xyz="0.0 0.0 0.0" rpy="0.0 0.0 0.0" />
         <geometry>
-          <mesh filename="package://ros_components_description/meshes/intel_realsense_d435.dae" />
+          <mesh filename="package://psd_sensors/meshes/intel_realsense_d435.dae" />
         </geometry>
       </visual>

File: urdf/luxonis_depthai.urdf.xacro (robot description, xacro)
@@ -16,5 +16,5 @@
 		cam_roll="${rpy.split()[0]}" cam_pitch="${rpy.split()[1]}" cam_yaw="${rpy.split()[2]}"
     simulation="${use_sim}" />
-  <xacro:include filename="$(find ros_components_description)/urdf/gz_sensor.urdf.xacro" ns="gz_sensor" />
+  <xacro:include filename="$(find psd_sensors)/urdf/gz_sensor.urdf.xacro" ns="gz_sensor" />
   <xacro:gz_sensor.camera
     reference="${ns}${device_namespace}"

File: urdf/orbbec_astra.urdf.xacro (robot description, xacro)
@@ -23,5 +23,5 @@
         <origin xyz="0.0 0.0 0.0" rpy="0.0 0.0 0.0" />
         <geometry>
-          <mesh filename="package://ros_components_description/meshes/orbbec_astra.dae" />
+          <mesh filename="package://psd_sensors/meshes/orbbec_astra.dae" />
         </geometry>
       </visual>
@@ -74,5 +74,5 @@
     <!-- GAZEBO -->
     <!-- https://github.com/orbbec/OrbbecSDK_ROS2#all-available-topics -->
-    <xacro:include filename="$(find ros_components_description)/urdf/gz_sensor.urdf.xacro" ns="gz_sensor" />
+    <xacro:include filename="$(find psd_sensors)/urdf/gz_sensor.urdf.xacro" ns="gz_sensor" />
     <xacro:gz_sensor.camera
       reference="${device_namespace}_link"

File: urdf/ouster.urdf.xacro (robot description, xacro)
@@ -55,5 +55,5 @@
         <origin xyz="0.0 0.0 0.0" rpy="0.0 0.0 0.0" />
         <geometry>
-          <mesh filename="package://ros_components_description/meshes/${mesh}.dae" />
+          <mesh filename="package://psd_sensors/meshes/${mesh}.dae" />
         </geometry>
       </visual>

File: urdf/slamtec_rplidar.urdf.xacro (robot description, xacro)
@@ -193,5 +193,5 @@
         <origin xyz="0.0 0.0 0.0" rpy="0.0 0.0 0.0" />
         <geometry>
-          <mesh filename="package://ros_components_description/meshes/rplidar/${mesh}" />
+          <mesh filename="package://psd_sensors/meshes/rplidar/${mesh}" />
         </geometry>
       </visual>

File: urdf/stereolabs_zed.urdf.xacro (robot description, xacro)
@@ -86,5 +86,5 @@
         <origin xyz="${screw_offset_x} 0 ${screw_offset_z}" rpy="0 0 0" />
         <geometry>
-          <mesh filename="package://ros_components_description/meshes/${model}.stl" />
+          <mesh filename="package://psd_sensors/meshes/${model}.stl" />
         </geometry>
         <material name="mat">
@@ -94,5 +94,5 @@
       <collision>
         <geometry>
-          <mesh filename="package://ros_components_description/meshes/${model}.stl" />
+          <mesh filename="package://psd_sensors/meshes/${model}.stl" />
         </geometry>
       </collision>

File: urdf/teltonika_003R-00253.urdf.xacro (robot description, xacro)
@@ -18,5 +18,5 @@
         <origin xyz="0.0 0.0 0.0" rpy="0.0 0.0 0.0" />
         <geometry>
-          <mesh filename="package://ros_components_description/meshes/teltonika_003R-00253.dae" />
+          <mesh filename="package://psd_sensors/meshes/teltonika_003R-00253.dae" />
         </geometry>
       </visual>
@@ -25,5 +25,5 @@
         <geometry>
           <mesh
-            filename="package://ros_components_description/meshes/teltonika_003R-00253_collision.stl" />
+            filename="package://psd_sensors/meshes/teltonika_003R-00253_collision.stl" />
         </geometry>
       </collision>

File: urdf/ur.urdf.xacro (robot description, xacro)
@@ -33,5 +33,5 @@
       value="$(find ur_description)/config/${ur_type}/visual_parameters.yaml" scope="parent" />
     <xacro:property name="simulation_controllers"
-      value="$(find ros_components_description)/config/ur_controllers.yaml" scope="parent" />
+      value="$(find psd_sensors)/config/ur_controllers.yaml" scope="parent" />
       <xacro:property name="initial_positions_file" default="$(find ur_description)/config/initial_positions.yaml" />
       <xacro:property name="initial_positions"

File: urdf/velodyne_puck.urdf.xacro (robot description, xacro)
@@ -18,5 +18,5 @@
         <origin xyz="0.0 0.0 0.0" rpy="0.0 0.0 0.0" />
         <geometry>
-          <mesh filename="package://ros_components_description/meshes/velodyne_puck.dae" />
+          <mesh filename="package://psd_sensors/meshes/velodyne_puck.dae" />
         </geometry>
       </visual>

File: urdf/wibotic_receiver.urdf.xacro (robot description, xacro)
@@ -33,5 +33,5 @@
         <origin xyz="0.0 0.0 0.0" rpy="0.0 0.0 ${pi/2.0}" />
         <geometry>
-          <mesh filename="package://ros_components_description/meshes/wibotic_receiver.stl" />
+          <mesh filename="package://psd_sensors/meshes/wibotic_receiver.stl" />
         </geometry>
         <material name="Grey">
@@ -42,5 +42,5 @@
         <origin xyz="0.0 0.0 0.0" rpy="0.0 0.0 ${pi/2.0}" />
         <geometry>
-          <mesh filename="package://ros_components_description/meshes/wibotic_receiver.stl" />
+          <mesh filename="package://psd_sensors/meshes/wibotic_receiver.stl" />
         </geometry>
       </collision>

File: urdf/wibotic_station.urdf.xacro (robot description, xacro)
@@ -33,5 +33,5 @@
         <origin xyz="0.0 0.0 0.0" rpy="0.0 0.0 ${pi/2.0}" />
         <geometry>
-          <mesh filename="package://ros_components_description/meshes/wibotic_station.stl" />
+          <mesh filename="package://psd_sensors/meshes/wibotic_station.stl" />
         </geometry>
         <material name="LightGrey">
